File: hydrogen_sensors_board_v2.brd (EAGLE design)
At the start: 68.2 x 66 mm, 44 parts, among them U1 ATMEGA328P_TQFP, U2 TLV1117-33IDCY, Y1 16MHz

Commit message: changed a resistor value to a standard value
Parts:
- R13: value 40k -> 39k
Changed lines of the file:
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@@
 <?xml version="1.0" encoding="utf-8"?>
 <!DOCTYPE eagle SYSTEM "eagle.dtd">
-<eagle version="8.3.1">
+<eagle version="8.4.1">
 <drawing>
 <settings>
@@
 <param name="dpMaxLengthDifference" value="10mm"/>
 <param name="dpGapFactor" value="2.5"/>
-<param name="checkGrid" value="0"/>
 <param name="checkAngle" value="0"/>
 <param name="checkFont" value="1"/>
 <param name="checkRestrict" value="0"/>
+<param name="checkStop" value="0"/>
 <param name="useDiameter" value="13"/>
 <param name="maxErrors" value="50"/>
@@
 </element>
 <element name="R12" library="SparkFun-Passives" package="0603-RES" value="20k" x="51.816" y="25.4" rot="MR180"/>
-<element name="R13" library="SparkFun-Passives" package="0603-RES" value="40k" x="51.816" y="27.94" rot="MR0"/>
+<element name="R13" library="SparkFun-Passives" package="0603-RES" value="39k" x="51.816" y="27.94" rot="MR0"/>
 <element name="C11" library="adafruit" package="C0603" value="100nF" x="48.26" y="26.416" rot="MR0"/>
 <element name="E1" library="5555140-6 RJ11" package="1734723-1_RJ11" value="5555140-6" x="47.752" y="12.192"/>
